File: hardware/T568A_to_RJ11_adapter.kicad_sch (KiCad schematic)
At the start: 10 parts, among them J1 6P6C, J2 6P6C, J3 6P6C, J4 6P6C, J5 8P8C

Commit message: Update BOM and add photo of finished project.
Parts:
- J1, J2, J3, J4: Digi-Key_PN (none) -> 609-4729-ND; MPN (none) -> 54601-906WPLF
Changed lines of the file:
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@@
+			)
+		)
+		(property "MPN" "54601-906WPLF"
+			(at 140.97 66.04 90)
+			(effects
+				(font
+					(size 1.27 1.27)
+				)
+				(hide yes)
+			)
+		)
+		(property "Digi-Key_PN" "609-4729-ND"
+			(at 140.97 66.04 90)
+			(effects
+				(font
+					(size 1.27 1.27)
+				)
+				(hide yes)
 			)
 		)
@@
 			)
 		)
+		(property "MPN" "54601-906WPLF"
+			(at 166.37 66.04 90)
+			(effects
+				(font
+					(size 1.27 1.27)
+				)
+				(hide yes)
+			)
+		)
+		(property "Digi-Key_PN" "609-4729-ND"
+			(at 166.37 66.04 90)
+			(effects
+				(font
+					(size 1.27 1.27)
+				)
+				(hide yes)
+			)
+		)
 		(pin "5"
 		)
@@
 			)
 		)
+		(property "MPN" "54601-906WPLF"
+			(at 191.77 66.04 90)
+			(effects
+				(font
+					(size 1.27 1.27)
+				)
+				(hide yes)
+			)
+		)
+		(property "Digi-Key_PN" "609-4729-ND"
+			(at 191.77 66.04 90)
+			(effects
+				(font
+					(size 1.27 1.27)
+				)
+				(hide yes)
+			)
+		)
 		(pin "5"
 		)
@@
 			(effects
 				(font
+					(size 1.27 1.27)
+				)
+				(hide yes)
+			)
+		)
+		(property "Digi-Key_PN" "609-4729-ND"
+			(at 217.17 66.04 90)
+			(effects
+				(font
+					(size 1.27 1.27)
+				)
+				(hide yes)
+			)
+		)
+		(property "MPN" "54601-906WPLF"
+			(at 217.17 66.04 90)
+			(effects
+				(font
